Commit message: Updated robot_control.xacro in the src directory

File: src/description/urdf/robot_control.xacro (robot description, xacro)
@@ -3,41 +3,50 @@
 <xacro:macro name="control">
   <ros2_control name="SkidSteerSystem" type="system">
-  <hardware>
-    <plugin>gz_ros2_control/GazeboSimSystem</plugin>
-  </hardware>
-  <!-- Wheels -->
-  <joint name="front_left_wheel_joint">
-    <command_interface name="velocity"/>
-    <state_interface name="position"/>
-    <state_interface name="velocity"/>
-  </joint>
-  <joint name="rear_left_wheel_joint">
-    <command_interface name="velocity"/>
-    <state_interface name="position"/>
-    <state_interface name="velocity"/>
-  </joint>
-  <joint name="front_right_wheel_joint">
-    <command_interface name="velocity"/>
-    <state_interface name="position"/>
-    <state_interface name="velocity"/>
-  </joint>
-  <joint name="rear_right_wheel_joint">
-    <command_interface name="velocity"/>
-    <state_interface name="position"/>
-    <state_interface name="velocity"/>
-  </joint>
-  <!-- Turret PAN -->
-  <joint name="pan_joint">
-    <command_interface name="position"/>
-    <state_interface name="position"/>
-    <state_interface name="velocity"/>
-  </joint>
-  <!-- Turret TILT -->
-  <joint name="tilt_base_joint">
-    <command_interface name="position"/>
-    <state_interface name="position"/>
-    <state_interface name="velocity"/>
-  </joint>
-</ros2_control>
+    <hardware>
+      <plugin>gz_ros2_control/GazeboSimSystem</plugin>
+    </hardware>
+    <!-- ── SUSPENSION JOINTS (passive differential rocker) ───────────
+    ──────────────────────────────────────────────────────────────── -->
+    <joint name="left_suspension_joint">
+      <state_interface name="position"/>
+      <state_interface name="velocity"/>
+    </joint>
+    <joint name="right_suspension_joint">
+      <state_interface name="position"/>
+      <state_interface name="velocity"/>
+    </joint>
+    <!-- ── DRIVE WHEELS ─────────────────────────────────────────── -->
+    <joint name="front_left_wheel_joint">
+      <command_interface name="velocity"/>
+      <state_interface  name="position"/>
+      <state_interface  name="velocity"/>
+    </joint>
+    <joint name="rear_left_wheel_joint">
+      <command_interface name="velocity"/>
+      <state_interface  name="position"/>
+      <state_interface  name="velocity"/>
+    </joint>
+    <joint name="front_right_wheel_joint">
+      <command_interface name="velocity"/>
+      <state_interface  name="position"/>
+      <state_interface  name="velocity"/>
+    </joint>
+    <joint name="rear_right_wheel_joint">
+      <command_interface name="velocity"/>
+      <state_interface  name="position"/>
+      <state_interface  name="velocity"/>
+    </joint>
+    <!-- ── TURRET ────────────────────────────────────────────────── -->
+    <joint name="pan_joint">
+      <command_interface name="position"/>
+      <state_interface  name="position"/>
+      <state_interface  name="velocity"/>
+    </joint>
+    <joint name="tilt_base_joint">
+      <command_interface name="position"/>
+      <state_interface  name="position"/>
+      <state_interface  name="velocity"/>
+    </joint>
+  </ros2_control>
 </xacro:macro>
 </robot>
