Commit message: Updated the URDF with the real CAD meshes

File: src/description/urdf/robot_base.xacro (robot description, xacro)
@@ -2,30 +2,39 @@
 <robot xmlns:xacro="http://www.ros.org/wiki/xacro">
   <xacro:macro name="base">
-    <xacro:property name="base_length" value="0.5"/>
-    <xacro:property name="base_width" value="0.4"/>
-    <xacro:property name="base_height" value="0.2"/>
-    <xacro:property name="wheel_radius" value="0.075"/>
-    <xacro:property name="wheel_width" value="0.04"/>
-    <xacro:property name="wheel_x_offset" value="0.18"/>
-    <xacro:property name="wheel_y_offset" value="0.22"/>
+    <xacro:property name="base_length" value="0.671"/>
+    <xacro:property name="base_width"  value="0.825"/>
+    <xacro:property name="base_height" value="0.266"/>
+    <xacro:property name="wheel_radius" value="0.155"/>
+    <xacro:property name="wheel_width"  value="0.162"/>
+    <xacro:property name="susp_pivot_x"  value="0.4291"/>
+    <xacro:property name="susp_pivot_z"  value="0.3130"/>
+    <xacro:property name="susp_left_y"   value="-0.266"/>
+    <xacro:property name="susp_right_y"  value=" 0.266"/>
+    <xacro:property name="susp_front_x"  value="0.546"/>
+    <xacro:property name="susp_front_y"  value="-0.066"/>
+    <xacro:property name="susp_front_z"  value="-0.389"/>
+    <xacro:property name="susp_rear_x"   value="-0.609"/>
+    <xacro:property name="susp_rear_y"   value="-0.068"/>
+    <xacro:property name="susp_rear_z"   value="-0.278"/>
+    <!-- ══════════════════════════════════════════════════════════════
+         BASE LINK
+         ══════════════════════════════════════════════════════════════ -->
     <link name="base_link">
       <visual>
+        <origin xyz="0.0709 0.0709 0.0267" rpy="1.5708 0 1.5708"/>
         <geometry>
-          <box size="${base_length} ${base_width} ${base_height}"/>
+          <mesh filename="file://$(find description)/meshes/chassis.dae"
+                scale="0.001 0.001 0.001"/>
         </geometry>
-        <origin xyz="0 0 ${base_height/2}" rpy="0 0 0"/>
-        <material name="body_color">
-          <color rgba="0.15 0.15 0.18 1"/>
-        </material>
       </visual>
       <collision>
         <geometry>
-          <box size="${base_length} ${base_width} ${base_height}"/>
+          <box size="${base_width} ${base_length} ${base_height}"/>
         </geometry>
-        <origin xyz="0 0 ${base_height/2}" rpy="0 0 0"/>
+        <origin xyz="0 0 ${wheel_radius*2 + base_height/2}" rpy="0 0 0"/>
       </collision>
       <inertial>
         <mass value="10.0"/>
-        <origin xyz="0 0 ${base_height/2}"/>
+        <origin xyz="0 0 ${wheel_radius*2 + base_height/2}"/>
         <inertia ixx="0.2" iyy="0.2" izz="0.2" ixy="0" ixz="0" iyz="0"/>
       </inertial>
@@ -34,178 +43,82 @@
       <self_collide>false</self_collide>
     </gazebo>
-    <link name="imu_link">
-      <visual>
-        <geometry>
-          <box size="0.03 0.03 0.02"/>
-        </geometry>
-        <origin xyz="0 0 0"/>
-        <material name="orange">
-          <color rgba="1 0.5 0 1"/>
-        </material>
-      </visual>
-    </link>
-    <joint name="imu_joint" type="fixed">
-      <parent link="base_link"/>
-      <child link="imu_link"/>
-      <origin xyz="0 0 0.15"/>
-    </joint>
-    <link name="gps_link">
-      <visual>
-        <geometry>
-          <box size="0.03 0.03 0.02"/>
-        </geometry>
-        <origin xyz="0 0 0"/>
-        <material name="white">
-          <color rgba="1 1 1 1"/>
-        </material>
-      </visual>
-    </link>
-    <joint name="gps_joint" type="fixed">
-      <parent link="base_link"/>
-      <child link="gps_link"/>
-      <origin xyz="0 0 0.2"/>
-    </joint>
-    <link name="lidar_link">
-      <visual>
-        <geometry>
-          <cylinder radius="0.04" length="0.05"/>
-        </geometry>
-        <origin xyz="0 0 0"/>
-        <material name="gray">
-          <color rgba="0.6 0.6 0.6 1.0"/>
-        </material>
-      </visual>
-      <collision>
-        <geometry>
-          <cylinder radius="0.04" length="0.05"/>
-        </geometry>
-        <origin xyz="0 0 0"/>
-      </collision>
-    </link>
-    <joint name="lidar_joint" type="fixed">
-      <parent link="base_link"/>
-      <child link="lidar_link"/>
-      <origin xyz="0.22 0 0.22"/>
-    </joint>
-    <!-- ================= PAN LINK ================= -->
-<link name="pan_link">
-  <visual>
-    <geometry>
-      <cylinder radius="0.05" length="0.02"/>
-    </geometry>
-    <material name="red">
-      <color rgba="1 0 0 1"/>
-    </material>
-  </visual>
-  <collision>
-    <geometry>
-      <cylinder radius="0.05" length="0.02"/>
-    </geometry>
-  </collision>
-  <inertial>
-    <mass value="0.5"/>
-    <origin xyz="0 0 0"/>
-    <inertia ixx="0.01" iyy="0.01" izz="0.01"
-             ixy="0" ixz="0" iyz="0"/>
-  </inertial>
-</link>
-<joint name="pan_joint" type="revolute">
-  <parent link="base_link"/>
-  <child link="pan_link"/>
-  <origin xyz="0.12 0 0.21"/>
-  <axis xyz="0 0 1"/>
-  <limit lower="-3.14" upper="3.14" effort="5" velocity="1"/>
-  <dynamics damping="0.1" friction="0.1"/>
-</joint>
-<!-- ================= TILT LINK ================= -->
-<link name="tilt_link">
-  <visual>
-    <geometry>
-      <box size="0.04 0.04 0.02"/>
-    </geometry>
-    <material name="black">
-      <color rgba="0.1 0.1 0.1 1"/>
-    </material>
-  </visual>
-  <collision>
-    <geometry>
-      <box size="0.04 0.04 0.02"/>
-    </geometry>
-  </collision>
-  <inertial>
-    <mass value="0.3"/>
-    <origin xyz="0 0 0"/>
-    <inertia ixx="0.005" iyy="0.005" izz="0.005"
-             ixy="0" ixz="0" iyz="0"/>
-  </inertial>
-</link>
-<joint name="tilt_base_joint" type="revolute">
-  <parent link="pan_link"/>
-  <child link="tilt_link"/>
-  <origin xyz="0 0 0.05"/>
-  <axis xyz="0 1 0"/>
-  <limit lower="-1.57" upper="1.57" effort="5" velocity="1"/>
-  <dynamics damping="0.1" friction="0.1"/>
-</joint>
-<!-- ================= TURRET CAMERA ================= -->
-<link name="turret_camera_link">
-  <visual>
-    <geometry>
-      <box size="0.05 0.05 0.05"/>
-    </geometry>
-    <material name="Red">
-      <color rgba="1 0 0 1"/>
-    </material>
-  </visual>
-  <collision>
-    <geometry>
-      <box size="0.05 0.05 0.05"/>
-    </geometry>
-  </collision>
-  <inertial>
-    <mass value="0.3"/>
-    <origin xyz="0 0 0"/>
-    <inertia ixx="0.005" iyy="0.005" izz="0.005"
-             ixy="0" ixz="0" iyz="0"/>
-  </inertial>
-</link>
-<joint name="turret_camera_joint" type="fixed">
-  <parent link="tilt_link"/>
-  <child link="turret_camera_link"/>
-  <origin xyz="0 0 0.03"/>
-</joint>
-<!-- ================= LANE CAMERA ================= -->
-<link name="camera_link">
-  <visual>
-    <geometry>
-      <box size="0.05 0.05 0.05"/>
-    </geometry>
-    <material name="blue">
-      <color rgba="0 0 1 1"/>
-    </material>
-  </visual>
-  <collision>
-    <geometry>
-      <box size="0.05 0.05 0.05"/>
-    </geometry>
-  </collision>
-  <inertial>
-    <mass value="0.3"/>
-    <origin xyz="0 0 0"/>
-    <inertia ixx="0.005" iyy="0.005" izz="0.005"
-             ixy="0" ixz="0" iyz="0"/>
-  </inertial>
-</link>
-<joint name="camera_joint" type="fixed">
-  <parent link="base_link"/>
-  <child link="camera_link"/>
-  <origin xyz="0.15 0 1" rpy="0 0.25 0"/> <!-- chcanged camera and turret positions-->
-</joint>
-    <xacro:macro name="wheel" params="name x y">
+    <!-- ══════════════════════════════════════════════════════════════
+         SUSPENSION MACRO
+         ══════════════════════════════════════════════════════════════ -->
+    <xacro:macro name="suspension_arm" params="side pivot_y">
+      <link name="${side}_suspension_link">
+        <visual>
+          <origin xyz="-0.356 0.147 -0.211" rpy="1.5708 0 0"/>
+          <geometry>
+            <mesh filename="file://$(find description)/meshes/suspension.dae"
+                  scale="0.001 0.001 0.001"/>
+          </geometry>
+        </visual>
+        <collision>
+          <geometry><box size="1.2 0.1 0.15"/></geometry>
+          <origin xyz="0 0 0" rpy="0 0 0"/>
+        </collision>
+        <inertial>
+          <mass value="2.0"/>
+          <origin xyz="0 0 0"/>
+          <inertia ixx="0.005" iyy="0.240" izz="0.240"
+                   ixy="0"     ixz="0"     iyz="0"/>
+        </inertial>
+      </link>
+      <gazebo reference="${side}_suspension_link">
+        <self_collide>false</self_collide>
+      </gazebo>
+    </xacro:macro>
+    <!-- ── LEFT suspension joint ─────────────────────────────────────
+         This is the FREE joint — terrain forces drive it passively.
+         No command interface. gz_ros2_control reads this to compute
+         the right joint position every physics tick.
+    ─────────────────────────────────────────────────────────────────── -->
+    <xacro:suspension_arm side="left" pivot_y="${susp_left_y}"/>
+    <joint name="left_suspension_joint" type="revolute">
+      <parent link="base_link"/>
+      <child  link="left_suspension_link"/>
+      <origin xyz="${susp_pivot_x} ${susp_left_y} ${susp_pivot_z}" rpy="0 0 0"/>
+      <axis xyz="0 1 0"/>
+      <limit lower="-1.047" upper="1.047" effort="0" velocity="1.0"/>
+      <dynamics damping="0.5" friction="0.1"/>
+    </joint>
+    <!-- ── RIGHT suspension joint ────────────────────────────────────
+         MIMIC joint. Follows left with multiplier -1.0:
+           right_angle = left_angle × -1.0
+         This enforces the differential rocker behaviour:
+           left arm tilts forward → right arm tilts backward
+         effort="0": passive, no motor.
+         gz_ros2_control reads the <mimic> tag and enforces it in
+         the physics engine every simulation tick.
+    ─────────────────────────────────────────────────────────────────── -->
+    <xacro:suspension_arm side="right" pivot_y="${susp_right_y}"/>
+    <joint name="right_suspension_joint" type="revolute">
+      <parent link="base_link"/>
+      <child  link="right_suspension_link"/>
+      <origin xyz="${susp_pivot_x} ${susp_right_y} ${susp_pivot_z}" rpy="0 0 0"/>
+      <axis xyz="0 1 0"/>
+      <limit lower="-1.047" upper="1.047" effort="0" velocity="1.0"/>
+      <dynamics damping="0.5" friction="0.1"/>
+      <!-- ═══ DIFFERENTIAL ROCKER CONSTRAINT ═══
+           right = left × -1.0
+           Enforced visually by robot_state_publisher (RViz).
+           Enforced in physics by gz_ros2_control GazeboSimSystem
+           (no separate plugin needed for Gazebo Ignition + Jazzy). -->
+      <mimic joint="left_suspension_joint" multiplier="-1.0" offset="0"/>
+    </joint>
+    <!-- ══════════════════════════════════════════════════════════════
+         WHEEL MACRO
+         ── vis_rpy parameter controls which face points outward ──────
+           left  wheels : vis_rpy="1.5708 0 0"        (unchanged)
+           right wheels : vis_rpy="1.5708 0 3.14159"  (Rz 180° flip)
+         ══════════════════════════════════════════════════════════════ -->
+    <xacro:macro name="wheel" params="name parent x y z vis_rpy">
       <link name="${name}_link">
         <visual>
-          <origin rpy="1.5708 0 0"/>
+          <origin rpy="${vis_rpy}"/>
           <geometry>
-            <cylinder radius="${wheel_radius}" length="${wheel_width}"/>
+            <mesh filename="file://$(find description)/meshes/wheel.dae"
+                  scale="0.001 0.001 0.001"/>
           </geometry>
           <material name="black">
@@ -214,7 +127,8 @@
         </visual>
         <collision>
-          <origin rpy="1.5708 0 0"/>
+          <origin rpy="${vis_rpy}"/>
           <geometry>
-            <cylinder radius="${wheel_radius}" length="${wheel_width}"/>
+            <mesh filename="file://$(find description)/meshes/wheel.dae"
+                  scale="0.001 0.001 0.001"/>
           </geometry>
         </collision>
@@ -222,26 +136,168 @@
           <mass value="1.0"/>
           <origin xyz="0 0 0"/>
-          <inertia ixx="0.01" iyy="0.01" izz="0.005" ixy="0" ixz="0" iyz="0"/>
+          <inertia ixx="0.010" iyy="0.010" izz="0.012"
+                   ixy="0"     ixz="0"     iyz="0"/>
         </inertial>
       </link>
       <joint name="${name}_joint" type="continuous">
-        <parent link="base_link"/>
-        <child link="${name}_link"/>
-        <origin xyz="${x} ${y} ${wheel_radius}"/>
+        <parent link="${parent}"/>
+        <child  link="${name}_link"/>
+        <origin xyz="${x} ${y} ${z}" rpy="0 0 0"/>
         <axis xyz="0 1 0"/>
+        <dynamics damping="0.01" friction="0.1"/>
       </joint>
+      <gazebo reference="${name}_link">
+        <mu1>0.8</mu1>
+        <mu2>0.8</mu2>
+        <self_collide>false</self_collide>
+      </gazebo>
     </xacro:macro>
+    <!-- Left  wheels : vis_rpy unchanged "1.5708 0 0" -->
     <xacro:wheel name="front_left_wheel"
-                 x="${wheel_x_offset}"
-                 y="${wheel_y_offset}"/>
+                 parent="left_suspension_link"
+                 x="${susp_front_x}" y="${susp_front_y}" z="${susp_front_z}"
+                 vis_rpy="1.5708 0 0"/>
     <xacro:wheel name="rear_left_wheel"
-                 x="-${wheel_x_offset}"
-                 y="${wheel_y_offset}"/>
+                 parent="left_suspension_link"
+                 x="${susp_rear_x}" y="${susp_rear_y}" z="${susp_rear_z}"
+                 vis_rpy="1.5708 0 0"/>
+    <!-- Right wheels : Rz 180° flips the outer face to point outward -->
     <xacro:wheel name="front_right_wheel"
-                 x="${wheel_x_offset}"
-                 y="-${wheel_y_offset}"/>
+                 parent="right_suspension_link"
+                 x="${susp_front_x}" y="${-susp_front_y}" z="${susp_front_z}"
+                 vis_rpy="1.5708 0 3.14159"/>
     <xacro:wheel name="rear_right_wheel"
-                 x="-${wheel_x_offset}"
-                 y="-${wheel_y_offset}"/>
+                 parent="right_suspension_link"
+                 x="${susp_rear_x}" y="${-susp_rear_y}" z="${susp_rear_z}"
+                 vis_rpy="1.5708 0 3.14159"/>
+    <!-- ═══════════ IMU ═══════════ -->
+    <link name="imu_link">
+      <visual>
+        <geometry><box size="0.03 0.03 0.02"/></geometry>
+        <origin xyz="0 0 0"/>
+        <material name="orange"><color rgba="1 0.5 0 1"/></material>
+      </visual>
+    </link>
+    <joint name="imu_joint" type="fixed">
+      <parent link="base_link"/>
+      <child  link="imu_link"/>
+      <origin xyz="0 0 0.15"/>
+    </joint>
+    <!-- ═══════════ GPS ═══════════ -->
+    <link name="gps_link">
+      <visual>
+        <geometry><box size="0.03 0.03 0.02"/></geometry>
+        <origin xyz="0 0 0"/>
+        <material name="white"><color rgba="1 1 1 1"/></material>
+      </visual>
+    </link>
+    <joint name="gps_joint" type="fixed">
+      <parent link="base_link"/>
+      <child  link="gps_link"/>
+      <origin xyz="0 0 0.2"/>
+    </joint>
+    <!-- ═══════════ LIDAR ═══════════ -->
+    <link name="lidar_link">
+      <visual>
+        <geometry><cylinder radius="0.04" length="0.05"/></geometry>
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
Commit message: Tweaked robot_xacro acc to the changes in robot_base

File: src/description/urdf/robot_base.xacro (robot description, xacro)
@@ -71,7 +71,4 @@
     </xacro:macro>
     <!-- ── LEFT suspension joint ─────────────────────────────────────
-         This is the FREE joint — terrain forces drive it passively.
-         No command interface. gz_ros2_control reads this to compute
-         the right joint position every physics tick.
     ─────────────────────────────────────────────────────────────────── -->
     <xacro:suspension_arm side="left" pivot_y="${susp_left_y}"/>
@@ -88,8 +85,4 @@
            right_angle = left_angle × -1.0
          This enforces the differential rocker behaviour:
-           left arm tilts forward → right arm tilts backward
-         effort="0": passive, no motor.
-         gz_ros2_control reads the <mimic> tag and enforces it in
-         the physics engine every simulation tick.
     ─────────────────────────────────────────────────────────────────── -->
     <xacro:suspension_arm side="right" pivot_y="${susp_right_y}"/>
@@ -101,9 +94,4 @@
       <limit lower="-1.047" upper="1.047" effort="0" velocity="1.0"/>
       <dynamics damping="0.5" friction="0.1"/>
-      <!-- ═══ DIFFERENTIAL ROCKER CONSTRAINT ═══
-           right = left × -1.0
-           Enforced visually by robot_state_publisher (RViz).
-           Enforced in physics by gz_ros2_control GazeboSimSystem
-           (no separate plugin needed for Gazebo Ignition + Jazzy). -->
       <mimic joint="left_suspension_joint" multiplier="-1.0" offset="0"/>
     </joint>
@@ -111,6 +99,6 @@
          WHEEL MACRO
          ── vis_rpy parameter controls which face points outward ──────
-           left  wheels : vis_rpy="1.5708 0 0"        (unchanged)
-           right wheels : vis_rpy="1.5708 0 3.14159"  (Rz 180° flip)
+           left  wheels : vis_rpy="1.5708 0 0"
+           right wheels : vis_rpy="1.5708 0 3.14159"
          ══════════════════════════════════════════════════════════════ -->
     <xacro:macro name="wheel" params="name parent x y z vis_rpy">
@@ -153,5 +141,5 @@
       </gazebo>
     </xacro:macro>
-    <!-- Left  wheels : vis_rpy unchanged "1.5708 0 0" -->
+    <!-- Left  wheels -->
     <xacro:wheel name="front_left_wheel"
                  parent="left_suspension_link"
@@ -162,5 +150,5 @@
                  x="${susp_rear_x}" y="${susp_rear_y}" z="${susp_rear_z}"
                  vis_rpy="1.5708 0 0"/>
-    <!-- Right wheels : Rz 180° flips the outer face to point outward -->
+    <!-- Right wheels -->
     <xacro:wheel name="front_right_wheel"
                  parent="right_suspension_link"

Commit message: Updated robot_base.xacro for proper orientation

File: src/description/urdf/robot_base.xacro (robot description, xacro)
@@ -19,4 +19,8 @@
     <!-- ══════════════════════════════════════════════════════════════
          BASE LINK
+         base_link origin = chassis centre (midpoint of body).
+         Lowest point (front wheel bottom) = susp_pivot_z + susp_front_z - wheel_radius
+                                           = 0.313 - 0.389 - 0.155 = -0.231 m
+         → spawn the robot at z ≥ 0.25 in your launch file.
          ══════════════════════════════════════════════════════════════ -->
     <link name="base_link">
@@ -32,9 +36,11 @@
           <box size="${base_width} ${base_length} ${base_height}"/>
         </geometry>
-        <origin xyz="0 0 ${wheel_radius*2 + base_height/2}" rpy="0 0 0"/>
+        <!-- Centred at base_link origin (chassis midpoint) -->
+        <origin xyz="0 0 0" rpy="0 0 0"/>
       </collision>
       <inertial>
         <mass value="10.0"/>
-        <origin xyz="0 0 ${wheel_radius*2 + base_height/2}"/>
+        <!-- CoM at chassis centre -->
+        <origin xyz="0 0 0"/>
         <inertia ixx="0.2" iyy="0.2" izz="0.2" ixy="0" ixz="0" iyz="0"/>
       </inertial>
@@ -56,5 +62,5 @@
         </visual>
         <collision>
-          <geometry><box size="1.2 0.1 0.15"/></geometry>
+          <geometry><box size="0.01 0.01 0.01"/></geometry>
           <origin xyz="0 0 0" rpy="0 0 0"/>
         </collision>
@@ -70,6 +76,5 @@
       </gazebo>
     </xacro:macro>
-    <!-- ── LEFT suspension joint ─────────────────────────────────────
-    ─────────────────────────────────────────────────────────────────── -->
+    <!-- ── LEFT suspension ───────────────────────────────────────── -->
     <xacro:suspension_arm side="left" pivot_y="${susp_left_y}"/>
     <joint name="left_suspension_joint" type="revolute">
@@ -81,9 +86,5 @@
       <dynamics damping="0.5" friction="0.1"/>
     </joint>
-    <!-- ── RIGHT suspension joint ────────────────────────────────────
-         MIMIC joint. Follows left with multiplier -1.0:
-           right_angle = left_angle × -1.0
-         This enforces the differential rocker behaviour:
-    ─────────────────────────────────────────────────────────────────── -->
+    <!-- ── RIGHT suspension (mimic) ─────────────────────────────── -->
     <xacro:suspension_arm side="right" pivot_y="${susp_right_y}"/>
     <joint name="right_suspension_joint" type="revolute">
@@ -98,7 +99,4 @@
     <!-- ══════════════════════════════════════════════════════════════
          WHEEL MACRO
-         ── vis_rpy parameter controls which face points outward ──────
-           left  wheels : vis_rpy="1.5708 0 0"
-           right wheels : vis_rpy="1.5708 0 3.14159"
          ══════════════════════════════════════════════════════════════ -->
     <xacro:macro name="wheel" params="name parent x y z vis_rpy">
@@ -136,6 +134,8 @@
       </joint>
       <gazebo reference="${name}_link">
-        <mu1>0.8</mu1>
-        <mu2>0.8</mu2>
+        <mu1>2.0</mu1>
+        <mu2>2.0</mu2>
+        <kp>1e6</kp>
+        <kd>1.0</kd>
         <self_collide>false</self_collide>
       </gazebo>
