Commit message: Add mercury custom driver, drive controller, configurations, and test scripts

File: src/description/urdf/robot_base.xacro (robot description, xacro)
@@ -34,8 +34,8 @@
       <collision>
         <geometry>
-          <box size="${base_width} ${base_length} ${base_height}"/>
+          <box size="${base_width} 0.45 ${base_height}"/>
         </geometry>
-        <!-- Centred at base_link origin (chassis midpoint) -->
-        <origin xyz="0 0 0" rpy="0 0 0"/>
+        <!-- Offset upwards to avoid ground scraping and provide ground clearance -->
+        <origin xyz="0 0 0.05" rpy="0 0 0"/>
       </collision>
       <inertial>
@@ -83,6 +83,6 @@
       <origin xyz="${susp_pivot_x} ${susp_left_y} ${susp_pivot_z}" rpy="0 0 0"/>
       <axis xyz="0 1 0"/>
-      <limit lower="-1.047" upper="1.047" effort="0" velocity="1.0"/>
-      <dynamics damping="0.5" friction="0.1"/>
+      <limit lower="0.0" upper="0.0" effort="0" velocity="0.0"/>
+      <dynamics damping="10.0" friction="10.0"/>
     </joint>
     <!-- ── RIGHT suspension (mimic) ─────────────────────────────── -->
@@ -93,6 +93,6 @@
       <origin xyz="${susp_pivot_x} ${susp_right_y} ${susp_pivot_z}" rpy="0 0 0"/>
       <axis xyz="0 1 0"/>
-      <limit lower="-1.047" upper="1.047" effort="0" velocity="1.0"/>
-      <dynamics damping="0.5" friction="0.1"/>
+      <limit lower="0.0" upper="0.0" effort="0" velocity="0.0"/>
+      <dynamics damping="10.0" friction="10.0"/>
       <mimic joint="left_suspension_joint" multiplier="-1.0" offset="0"/>
     </joint>
@@ -134,6 +134,7 @@
       </joint>
       <gazebo reference="${name}_link">
-        <mu1>2.0</mu1>
-        <mu2>2.0</mu2>
+        <mu1>10.0</mu1>
+        <mu2>0.05</mu2>
+        <fdir1>1 0 0</fdir1>
         <kp>1e6</kp>
         <kd>1.0</kd>

File: src/description/urdf/robot_control.xacro (robot description, xacro)
@@ -12,5 +12,13 @@
       <state_interface name="velocity"/>
     </joint>
+    <!-- right_suspension_joint mirrors left at -1× via gz_ros2_control software mimic.
+         This is the correct fix for Gazebo Harmonic / ROS2 Jazzy because the default
+         DART physics engine does NOT support native mimic constraints at the physics
+         level. gz_ros2_control reads the <param name="mimic"> tag and enforces the
+         coupling in the control layer instead. -->
     <joint name="right_suspension_joint">
+      <param name="mimic">left_suspension_joint</param>
+      <param name="multiplier">-1.0</param>
+      <param name="offset">0.0</param>
       <state_interface name="position"/>
       <state_interface name="velocity"/>

Commit message: Update rover chassis color and materials

File: src/description/urdf/robot_base.xacro (robot description, xacro)
@@ -31,4 +31,7 @@
                 scale="0.001 0.001 0.001"/>
         </geometry>
+       <material name="yellow_body">
+           <colour rgba="1.0 1.0 0.0 1.0"/>
+       </material>
       </visual>
       <collision>
@@ -47,4 +50,5 @@
     </link>
     <gazebo reference="base_link">
+      <material>Gazebo/Yellow</material>
       <self_collide>false</self_collide>
     </gazebo>
@@ -109,5 +113,5 @@
           </geometry>
           <material name="black">
-            <color rgba="0.05 0.05 0.05 1"/>
+            <color rgba="0.5 0.0 1.0 1.0"/>
           </material>
         </visual>
@@ -165,5 +169,5 @@
         <geometry><box size="0.03 0.03 0.02"/></geometry>
         <origin xyz="0 0 0"/>
-        <material name="orange"><color rgba="1 0.5 0 1"/></material>
+        <material name="orange"><color rgba="0.5 0.0 1.0 1.0"/></material>
       </visual>
     </link>
@@ -178,5 +182,5 @@
         <geometry><box size="0.03 0.03 0.02"/></geometry>
         <origin xyz="0 0 0"/>
-        <material name="white"><color rgba="1 1 1 1"/></material>
+        <material name="white"><color rgba="0.5 0.0 1.0 1.0"/></material>
       </visual>
     </link>
@@ -191,5 +195,5 @@
         <geometry><cylinder radius="0.04" length="0.05"/></geometry>
         <origin xyz="0 0 0"/>
-        <material name="gray"><color rgba="0.6 0.6 0.6 1.0"/></material>
+        <material name="gray"><color rgba="0.5 0.0 1.0 1.0"/></material>
       </visual>
       <collision>
@@ -207,5 +211,5 @@
       <visual>
         <geometry><cylinder radius="0.05" length="0.02"/></geometry>
-        <material name="red"><color rgba="1 0 0 1"/></material>
+        <material name="red"><color rgba="0.5 0.0 1.0 1.0"/></material>
       </visual>
       <collision>
@@ -230,5 +234,5 @@
       <visual>
         <geometry><box size="0.04 0.04 0.02"/></geometry>
-        <material name="black"><color rgba="0.1 0.1 0.1 1"/></material>
+        <material name="black"><color rgba="0.5 0.0 1.0 1.0"/></material>
       </visual>
       <collision>
@@ -253,5 +257,5 @@
       <visual>
         <geometry><box size="0.05 0.05 0.05"/></geometry>
-        <material name="Red"><color rgba="1 0 0 1"/></material>
+        <material name="Red"><color rgba="0.5 0.0 1.0 1.0"/></material>
       </visual>
       <collision>
@@ -273,5 +277,5 @@
       <visual>
         <geometry><box size="0.05 0.05 0.05"/></geometry>
-        <material name="blue"><color rgba="0 0 1 1"/></material>
+        <material name="blue"><color rgba="0.5 0.0 1.0 1.0"/></material>
       </visual>
       <collision>
