Commit message: Port codebase to Ubuntu 22.04 (ROS 2 Humble / Ignition Fortress)
- Update Dockerfile and run.sh for ROS 2 Humble environment
- Configure ign_ros2_control hardware plugin and launch parameters
- Fix diff_drive_controller velocity topic relaying (/cmd_vel_unstamped)
- Resolve dual TF publishing conflict between diff_drive_controller and EKF
- Update Nav2 plugin naming conventions for Humble compatibility
- Fix RViz costmap display QoS durability policy (Volatile)
- Tune ODE physics solver and wheel contact surface friction
- Adjust base_link collision box to eliminate internal wheel overlap
- Add automated pre-launch process killer in simulation launch
- Add send_goal CLI utility for sending target coordinates from terminal

File: src/description/urdf/robot_base.xacro (robot description, xacro)
@@ -21,5 +21,5 @@
       <collision>
         <geometry>
-          <box size="${base_length} ${base_width} ${base_height}"/>
+          <box size="0.48 0.36 0.18"/>
         </geometry>
         <origin xyz="0 0 ${base_height/2 + wheel_radius}" rpy="0 0 0"/>
@@ -231,4 +231,13 @@
         <axis xyz="0 1 0"/>
       </joint>
+      <gazebo reference="${name}_link">
+        <self_collide>false</self_collide>
+        <mu1>0.8</mu1>
+        <mu2>0.8</mu2>
+        <kp>1000000.0</kp>
+        <kd>100.0</kd>
+        <minDepth>0.001</minDepth>
+        <maxVel>1.0</maxVel>
+      </gazebo>
     </xacro:macro>
     <xacro:wheel name="front_left_wheel"

File: src/description/urdf/robot_control.xacro (robot description, xacro)
@@ -4,5 +4,5 @@
   <ros2_control name="SkidSteerSystem" type="system">
   <hardware>
-    <plugin>gz_ros2_control/GazeboSimSystem</plugin>
+    <plugin>ign_ros2_control/IgnitionSystem</plugin>
   </hardware>
   <!-- Wheels -->

File: src/description/urdf/robot_sensors.xacro (robot description, xacro)
@@ -7,4 +7,7 @@
         <update_rate>100</update_rate>
         <topic>/imu</topic>
+        <ign_frame_id>imu_link</ign_frame_id>
+        <gz_frame_id>imu_link</gz_frame_id>
+        <frame_id>imu_link</frame_id>
       </sensor>
     </gazebo>
@@ -14,5 +17,7 @@
         <update_rate>5</update_rate>
         <topic>/gps</topic>
+        <ign_frame_id>gps_link</ign_frame_id>
         <gz_frame_id>gps_link</gz_frame_id>
+        <frame_id>gps_link</frame_id>
         <navsat>
           <position_sensing>
@@ -39,5 +44,7 @@
         <topic>/scan</topic>
         <visualize>true</visualize>
+        <ign_frame_id>lidar_link</ign_frame_id>
         <gz_frame_id>lidar_link</gz_frame_id>
+        <frame_id>lidar_link</frame_id>
         <lidar>
           <scan>
@@ -62,4 +69,7 @@
         <update_rate>30</update_rate>
         <topic>/camera/image_raw</topic>
+        <ign_frame_id>camera_link</ign_frame_id>
+        <gz_frame_id>camera_link</gz_frame_id>
+        <frame_id>camera_link</frame_id>
         <camera>
           <horizontal_fov>1.047</horizontal_fov>
@@ -81,4 +91,7 @@
     <update_rate>30</update_rate>
     <topic>/turret_camera/image_raw</topic>
+    <ign_frame_id>turret_camera_link</ign_frame_id>
+    <gz_frame_id>turret_camera_link</gz_frame_id>
+    <frame_id>turret_camera_link</frame_id>
     <camera>
       <horizontal_fov>1.047</horizontal_fov>

File: src/description/urdf/robot_sim.xacro (robot description, xacro)
@@ -3,6 +3,6 @@
   <xacro:macro name="sim">
     <gazebo>
-      <plugin filename="libgz_ros2_control-system.so"
-              name="gz_ros2_control::GazeboSimROS2ControlPlugin">
+      <plugin filename="libign_ros2_control-system.so"
+              name="ign_ros2_control::IgnitionROS2ControlPlugin">
         <parameters>$(find description)/config/controllers.yaml</parameters>
       </plugin>
